File: hardware/widebando2.kicad_pcb (KiCad board)
At the start: 2 copper layers, 110.5 x 60.2 mm, 21 parts, among them P1 CONN_9, P2 CONN_6, Q1 MOSFET_N, U1 TL082, U2 TL082, U3 78025

Commit message: Added labels
Routing:
- net Net-(P1-Pad6): track 18.0 -> 63.5 mm
- net +12V: track 153.5 -> 150.4 mm
- added copper zone on B.Cu, net GND
- added copper zone on F.Cu, net GND
Other:
- board text added: "AB1TJ DEC 2015 OXYGEN SENSOR CONTROLLER"
