File: hardware/widebando2.sch (KiCad schematic (older format))
At the start: 21 parts, among them P1 CONN_9, P2 CONN_6, Q1 MOSFET_N, U1 TL082, U2 TL082, U3 78025

Commit message: Added labels
Parts:
- P1: value CONN_9 -> MCU
- P2: value CONN_6 -> O2 Sensor
Other:
- note added: "HEATER CONTROL"
- note added: "IMPEDANCE\nPULSE GENERATION\n"
- note added: "IMPEDANCE\nPULSE MEASURE"
- note added: "MICROCONTROLLER\nCONNECTOR"
- note added: "PUMP CURRENT"
- note added: "REFERENCE\nGENERATION"
- note added: "SENSOR\nCONNECTOR"
Changed lines of the file:
@@
 LIBS:valves
 LIBS:78025
+LIBS:widebando2-cache
 EELAYER 25 0
 EELAYER END
@@
 P 1600 2750
 F 0 "P1" V 1550 2750 60  0000 C CNN
-F 1 "CONN_9" V 1650 2750 60  0000 C CNN
+F 1 "MCU" V 1650 2750 60  0000 C CNN
 F 2 "Terminal_Blocks:TerminalBlock_WAGO-804_RM5mm_9pol" H 1600 2750 60  0001 C CNN
 F 3 "" H 1600 2750 60  0000 C CNN
@@
 P 7300 2500
 F 0 "P2" V 7250 2500 60  0000 C CNN
-F 1 "CONN_6" V 7350 2500 60  0000 C CNN
+F 1 "O2 Sensor" V 7350 2500 60  0000 C CNN
 F 2 "Terminal_Blocks:TerminalBlock_WAGO-804_RM5mm_6pol" H 7300 2500 60  0001 C CNN
 F 3 "" H 7300 2500 60  0000 C CNN
@@
 	1    0    0    -1
 $EndComp
+Text Notes 3350 1850 0    60   ~ 12
+PUMP CURRENT
+Text Notes 4250 3250 0    60   ~ 12
+IMPEDANCE\nPULSE MEASURE
+Text Notes 5250 4250 0    60   ~ 12
+IMPEDANCE\nPULSE GENERATION\n
+Text Notes 3100 4700 0    60   ~ 12
+HEATER CONTROL
+Text Notes 1450 3150 1    60   ~ 12
+MICROCONTROLLER\nCONNECTOR
+Text Notes 7650 2250 3    60   ~ 12
+SENSOR\nCONNECTOR
+Text Notes 6250 2300 2    60   ~ 12
+REFERENCE\nGENERATION
 $EndSCHEMATC
